File: hardware/chufe-v-0-rev-a/chufe-v-0-rev-a.kicad_sch (KiCad schematic)
At the start: 0 parts

Commit message: agregar borrador sch
Parts:
- added C1, C2, C5: 100n, symbol Device:C
- added C3, C4: 10n, symbol Device:C
- added C6, C7: 1u, symbol Device:C_Polarized
- added C8: 10u, symbol Device:C_Polarized
- added D1, D2: D_Schottky, symbol Device:D_Schottky
- added J1: Conn_02x05_Odd_Even, symbol Connector_Generic:Conn_02x05_Odd_Even
- added J2, J3: AudioJack2_SwitchT, symbol Connector_Audio:AudioJack2_SwitchT
- added R1, R2, R3, R4: 1k, symbol Device:R
- added R5, R6: 100k, symbol Device:R
- added RV1, RV2: 100k, symbol Device:R_Potentiometer
- added U1: NE556, symbol Timer:NE556
Connections:
- new net: D1.2 (A), J1.10 (Pin_10), J1.9 (Pin_9)
- new net: R2.1, R4.1, U1.9 (OUT)
- new net: C7.1, R4.2
- new net: C1.1, RV1.3, U1.2 (THRES), U1.6 (TRIG)
- new net: R1.1, R3.1, U1.5 (OUT)
- new net: R1.2, RV1.1, RV1.2
- new net: C6.1, R3.2
- new net: D2.1 (K), J1.1 (Pin_1), J1.2 (Pin_2)
- new net: C7.2, J3.3, R6.2
- new net: C6.2, J2.3, R5.2
- new net: C2.1, RV2.3, U1.12 (THRES), U1.8 (TRIG)
- new net: C4.1, U1.11 (CONT)
- new net: R2.2, RV2.1, RV2.2
- new net: C3.1, U1.3 (CONT)
- new net +12V: C5.1, C8.1, D1.1 (K), U1.10 (~{RST}), U1.14 (VCC), U1.14 (VCC), U1.4 (~{RST})
- new net -12V: D2.2 (A)
- new net GND: C1.2, C2.2, C3.2, C4.2, C5.2, C8.2, J1.3 (Pin_3), J1.4 (Pin_4), J1.5 (Pin_5), J1.6 (Pin_6), J1.7 (Pin_7), J1.8 (Pin_8), J2.1, J3.1, R5.1, R6.1, U1.7 (GND), U1.7 (GND)
- no-connect marks 0 -> 4
Other:
- company: (none) -> piruetas SpA
- title: (none) -> cuadra-v0
