File: hardware/cuadra-v-0-rev-a/cuadra-v-0-rev-a.kicad_sch (KiCad schematic)
At the start: 22 parts, among them J1 Conn_02x05_Odd_Even, J2 AudioJack2_SwitchT, J3 AudioJack2_SwitchT, U1 NE556

Commit message: mejoras
Parts:
- removed C6, C7: 1u, symbol Device:C_Polarized
- removed D2: D_Schottky, symbol Device:D_Schottky
- added C6, C7: 1u, symbol Device:C
- added C9: 100n, symbol Device:C
Connections:
- net +12V: now also C9.1
- net GND: now also C9.2
- net at R4.2: now also C7.1
- net at R3.2: now also C6.1
- net at J3.3, R6.2: now also C7.2
- net at J2.3, R5.2: now also C6.2

Commit message: agregar entrada FM y resistor THT para afinar
Parts:
- added J1, J2: AudioJack2_SwitchT, symbol Connector_Audio:AudioJack2_SwitchT
- added R1: 100k, symbol Device:R
- added R2: 100k, Resistor_THT:R_Axial_DIN0207_L6.3mm_D2.5mm_P10.16mm_Horizontal, symbol Device:R
- C3, C4: value 10n -> 1n
- U1: value NE556 -> ICM7556; symbol Timer:NE556 -> Timer:ICM7556
- renumbered C9 to C5, C5 to C6, C8 to C7, C6 to C8, C7 to C9, J1 to J3, J2 to J4, J3 to J5, R1 to R3, R2 to R4, R3 to R5, R4 to R6, R5 to R7, R6 to R8
Connections:
- net GND: now also J1.1, J2.1
- net at C4.1, U1.11 (CONT): now also R2.2
- net at C3.1, U1.3 (CONT): now also R1.2
- new net: J1.3, R1.1
- new net: J2.3, R2.1
- no-connect marks 4 -> 6
Other:
- moved on the sheet: C1, C2, C3, C4, C5, C6, C7, C8, C9, D1, J3, J4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
